Commit message: add more joints and links

File: hpr_description/urdf/homeplater.urdf (robot description, URDF)
Before this commit: robot homeplater, 2 links, 1 joints
Links:
- added link left_wheel
Joints:
- added joint left_wheel_joint: type continuous, parent base_link, child left_wheel, origin xyz=0.048 0.095 0 rpy=1.571 0 0, axis 0 0 1
- joint caster joint: origin (none) -> xyz=-0.092 0 -0.0185 rpy=0.707 -0.707 -1.571

Commit message: finalize visual branch

File: hpr_description/urdf/homeplater.urdf (robot description, URDF)
Before this commit: robot homeplater, 3 links, 2 joints
Links:
- added link right_wheel; visual cylinder length=0.027 radius=0.0325
- link caster: geometry visual sphere radius=0.014
- link left_wheel: geometry visual cylinder length=0.027 radius=0.0325
Joints:
- added joint right_wheel_joint: type continuous, parent base_link, child right_wheel, origin xyz=0.048 -0.095 0 rpy=1.571 0 0, axis 0 0 1
- joint caster joint: origin xyz=-0.092 0 -0.0185 rpy=0.707 -0.707 -1.571 -> xyz=-0.044 0 -0.0185 rpy=0.707 -0.707 -1.571

Commit message: update readme

File: hpr_description/urdf/homeplater.urdf (robot description, URDF)
Before this commit: robot homeplater, 4 links, 3 joints
Joints:
- joint caster joint: origin xyz=-0.044 0 -0.0185 rpy=0.707 -0.707 -1.571 -> xyz=-0.044 0 -0.0315 rpy=0.707 -0.707 -1.571
- joint left_wheel_joint: origin xyz=0.048 0.095 0 rpy=1.571 0 0 -> xyz=0.048 0.095 -0.013 rpy=1.571 0 0
- joint right_wheel_joint: origin xyz=0.048 -0.095 0 rpy=1.571 0 0 -> xyz=0.048 -0.095 -0.013 rpy=1.571 0 0
