Commit message: update hpr urdf with multiple xacro

File: hpr_description/urdf/homeplater.urdf.xacro (robot description, xacro)
@@ -1,334 +1,4 @@
 <?xml version="1.0"?>
-<robot xmlns:xacro="http://www.ros.org/wiki/xacro" name="bot">
-    <!-- define colors -->
-    <material name="black">
-        <color rgba="0 0 0 1" />
-    </material>
-    <material name="white">
-        <color rgba="1 1 1 1" />
-    </material>
-    <material name="purple">
-        <color rgba="0.3098 0.1765 0.4980 1" />
-    </material>
-    <material name="orange">
-        <color rgba="1 0.6471 0 1" />
-    </material>
-    <material name="navy">
-        <color rgba="0 0 0.5 1" />
-    </material>
-    <material name="gray">
-        <color rgba="0.5 0.5 0.5 1" />
-    </material>
-    <!-- Define robot constants -->
-    <!-- pi -->
-    <xacro:property name="PI" value="3.141592653589793" />
-    <!-- base properties -->
-    <xacro:property name="base_width" value="0.4" />
-    <xacro:property name="base_depth" value="0.2" />
-    <xacro:property name="base_height" value="0.1" />
-    <xacro:property name="base_mass" value="2.0" />
-    <!-- wheel properties -->
-    <xacro:property name="wheel_ygap" value="0.005" />
-    <xacro:property name="wheel_xoff" value="0.1" />
-    <xacro:property name="wheel_radius" value="0.1" />
-    <xacro:property name="wheel_width" value="0.05" />
-    <xacro:property name="wheel_mass" value="0.2" />
-    <!-- caster properties -->
-    <xacro:property name="caster_xoff" value="-0.15" />
-    <xacro:property name="caster_radius" value="0.05" />
-    <xacro:property name="caster_mass" value="0.3" />
-    <!-- lidar properties -->
-    <xacro:property name="lidar_radius" value="0.035" />
-    <xacro:property name="lidar_height" value="0.02" />
-    <xacro:property name="lidar_zoff" value="0.05" />
-    <xacro:property name="lidar_mass" value="0.17" />
-    <!-- imu properties -->
-    <xacro:property name="imu_width" value="0.02" />
-    <xacro:property name="imu_depth" value="0.015" />
-    <xacro:property name="imu_height" value="0.001" />
-    <xacro:property name="imu_mass" value="0.002" />
-    <!-- Define intertial property macros  -->
-    <xacro:macro name="box_inertia" params="m w d h">
-        <inertial>
-            <origin xyz="0 0 0" rpy="${pi/2} 0 ${pi/2}" />
-            <mass value="${m}" />
-            <inertia ixx="${(m/12) * (h*h + d*d)}" ixy="0.0" ixz="0.0" iyy="${(m/12) * (w*w + h*h)}" iyz="0.0" izz="${(m/12) * (w*w + d*d)}" />
-        </inertial>
-    </xacro:macro>
-    <xacro:macro name="cylinder_inertia" params="m r h">
-        <inertial>
-            <origin xyz="0 0 0" rpy="${pi/2} 0 0" />
-            <mass value="${m}" />
-            <inertia ixx="${(m/12) * (3*r*r + h*h)}" ixy="0" ixz="0" iyy="${(m/12) * (3*r*r + h*h)}" iyz="0" izz="${(m/2) * (r*r)}" />
-        </inertial>
-    </xacro:macro>
-    <xacro:macro name="sphere_inertia" params="m r">
-        <inertial>
-            <mass value="${m}" />
-            <inertia ixx="${(2/5) * m * (r*r)}" ixy="0.0" ixz="0.0" iyy="${(2/5) * m * (r*r)}" iyz="0.0" izz="${(2/5) * m * (r*r)}" />
-        </inertial>
-    </xacro:macro>
-    <!-- Define wheel macros -->
-    <xacro:macro name="wheel" params="prefix y_reflect">
-        <joint name="${prefix}_joint" type="continuous">
-            <parent link="base_link" />
-            <child link="${prefix}_link" />
-            <origin xyz="${wheel_xoff} ${y_reflect*(base_depth/2+wheel_ygap+wheel_width/2)} 0" rpy="${-PI/2} 0 0" />
-            <axis xyz="0 0 1" />
-        </joint>
-        <link name="${prefix}_link">
-            <visual>
-                <geometry>
-                    <cylinder radius="${wheel_radius}" length="${wheel_width}" />
-                </geometry>
-                <material name="navy" />
-            </visual>
-            <collision>
-                <geometry>
-                    <cylinder radius="${wheel_radius}" length="${wheel_width}" />
-                </geometry>
-            </collision>
-            <xacro:cylinder_inertia m="${wheel_mass}" r="${wheel_radius}" h="${wheel_width}" />
-        </link>
-    </xacro:macro>
-    <!-- Robot Base -->
-    <link name="base_link">
-        <visual>
-            <geometry>
-                <box size="${base_width} ${base_depth} ${base_height}" />
-            </geometry>
-            <material name="orange" />
-        </visual>
-        <collision>
-            <geometry>
-                <box size="${base_width} ${base_depth} ${base_height}" />
-            </geometry>
-        </collision>
-    </link>
-    <gazebo reference="base_link">
-        <material>Gazebo/Wood</material>
-    </gazebo>
-    <!-- Robot Footprint -->
-    <joint name="footprint_joint" type="fixed">
-        <parent link="base_link" />
-        <child link="base_footprint" />
-        <origin xyz="0.0 0.0 ${-(wheel_radius)}" rpy="0 0 0" />
-    </joint>
-    <link name="base_footprint" />
-    <!-- Base Inertial -->
-    <joint name="base_inertial_joint" type="fixed">
-        <parent link="base_link" />
-        <child link="base_inertial" />
-        <origin xyz="0 0 0" rpy="0 0 0" />
-    </joint>
-    <link name="base_inertial">
-        <xacro:box_inertia m="${base_mass}" w="${base_width}" d="${base_depth}" h="${base_height}" />
-    </link>
-    <!-- Wheels -->
-    <xacro:wheel prefix="left_wheel" y_reflect="1" />
-    <gazebo reference="left_wheel_link">
-        <mu1>1.0</mu1>
-        <mu2>1.0</mu2>
-        <material>Gazebo/Blue</material>
-    </gazebo>
-    <xacro:wheel prefix="right_wheel" y_reflect="-1" />
-    <gazebo reference="right_wheel_link">
-        <mu1>1.0</mu1>
-        <mu2>1.0</mu2>
-        <material>Gazebo/Blue</material>
-    </gazebo>
-    <!-- Caster ball -->
-    <joint name="caster_joint" type="fixed">
-        <parent link="base_link" />
-        <child link="caster" />
-        <origin xyz="${caster_xoff} 0.0 ${-(base_height/2)}" rpy="0 0 0" />
-    </joint>
-    <link name="caster">
-        <visual>
-            <geometry>
-                <sphere radius="${caster_radius}" />
-            </geometry>
-            <material name="gray" />
-        </visual>
-        <collision>
-            <geometry>
-                <sphere radius="${caster_radius}" />
-            </geometry>
-        </collision>
-        <xacro:sphere_inertia m="${caster_mass}" r="${caster_radius}" />
-    </link>
-    <gazebo reference="caster">
-        <mu1>0.0</mu1>
-        <mu2>0.0</mu2>
-        <material>Gazebo/Gray</material>
-    </gazebo>
-    <!-- lidar -->
-    <joint name="lidar_joint" type="fixed">
-        <parent link="base_link" />
-        <child link="lidar_link" />
-        <origin xyz="0 0 ${(base_height+lidar_height)/2+lidar_zoff}" rpy="0 0 0" />
-    </joint>
-    <link name="lidar_link">
-        <visual>
-            <origin xyz="0 0 0" rpy="0 0 0" />
-            <geometry>
-                <cylinder radius="${lidar_radius}" length="${lidar_height}" />
-            </geometry>
-            <material name="black" />
-        </visual>
-        <collision>
-            <origin xyz="0 0 0" rpy="0 0 0" />
-            <geometry>
-                <cylinder radius="${lidar_radius}" length="${lidar_height}" />
-            </geometry>
-        </collision>
-        <xacro:cylinder_inertia m="${lidar_mass}" r="${lidar_radius}" h="${lidar_height}" />
-    </link>
-    <gazebo reference="lidar_link">
-        <material>Gazebo/Black</material>
-        <sensor name="lidar" type="ray">
-            <always_on>true</always_on>
-            <visualize>true</visualize>
-            <update_rate>5</update_rate>
-            <ray>
-                <scan>
-                    <horizontal>
-                        <samples>360</samples>
-                        <resolution>1.000000</resolution>
-                        <min_angle>0.000000</min_angle>
-                        <max_angle>6.280000</max_angle>
-                    </horizontal>
-                </scan>
-                <range>
-                    <min>0.120000</min>
-                    <max>6</max>
-                    <resolution>0.015000</resolution>
-                </range>
-                <noise>
-                    <type>gaussian</type>
-                    <mean>0.0</mean>
-                    <stddev>0.01</stddev>
-                </noise>
-            </ray>
-            <plugin name="scan" filename="libgazebo_ros_ray_sensor.so">
-                <ros>
-                    <remapping>~/out:=scan</remapping>
-                </ros>
-                <output_type>sensor_msgs/LaserScan</output_type>
-                <frame_name>lidar_link</frame_name>
-            </plugin>
-        </sensor>
-    </gazebo>
-    <!-- imu -->
-    <joint name="imu_joint" type="fixed">
-        <parent link="base_link"/>
-        <child link="imu_link"/>
-        <origin xyz="${base_width/4} 0 ${(base_height+imu_height)/2}"/>
-    </joint>
-    <link name="imu_link">
-        <visual>
-            <geometry>
-                <box size="${imu_width} ${imu_depth} ${imu_height}"/>
-            </geometry>
-            <material name="purple" />
-        </visual>
-        <collision>
-            <geometry>
-                <box size="${imu_width} ${imu_depth} ${imu_height}"/>
-            </geometry>
-        </collision>
-        <xacro:box_inertia m="${imu_mass}" w="${imu_width}" d="${imu_depth}" h="${imu_height}" />
-    </link>
-    <gazebo reference="imu_link">
-        <material>Gazebo/Purple</material>
-        <sensor name="imu_sensor" type="imu">
-            <plugin filename="libgazebo_ros_imu_sensor.so" name="imu_plugin">
-                <ros>
-                    <namespace>/bot</namespace>
-                    <remapping>~/out:=imu</remapping>
-                </ros>
-                <initial_orientation_as_reference>false</initial_orientation_as_reference>
-            </plugin>
-            <always_on>true</always_on>
-            <update_rate>100</update_rate>
-            <visualize>true</visualize>
-            <imu>
-                <angular_velocity>
-                    <x>
-                        <noise type="gaussian">
-                            <mean>0.0</mean>
-                            <stddev>2e-4</stddev>
-                            <bias_mean>0.0000075</bias_mean>
-                            <bias_stddev>0.0000008</bias_stddev>
-                        </noise>
-                    </x>
-                    <y>
-                        <noise type="gaussian">
-                            <mean>0.0</mean>
-                            <stddev>2e-4</stddev>
-                            <bias_mean>0.0000075</bias_mean>
-                            <bias_stddev>0.0000008</bias_stddev>
-                        </noise>
-                    </y>
-                    <z>
-                        <noise type="gaussian">
-                            <mean>0.0</mean>
-                            <stddev>2e-4</stddev>
-                            <bias_mean>0.0000075</bias_mean>
-                            <bias_stddev>0.0000008</bias_stddev>
-                        </noise>
-                    </z>
-                </angular_velocity>
-                <linear_acceleration>
-                    <x>
-                        <noise type="gaussian">
-                            <mean>0.0</mean>
-                            <stddev>1.7e-2</stddev>
-                            <bias_mean>0.1</bias_mean>
-                            <bias_stddev>0.001</bias_stddev>
-                        </noise>
-                    </x>
-                    <y>
-                        <noise type="gaussian">
-                            <mean>0.0</mean>
-                            <stddev>1.7e-2</stddev>
-                            <bias_mean>0.1</bias_mean>
-                            <bias_stddev>0.001</bias_stddev>
-                        </noise>
-                    </y>
-                    <z>
-                        <noise type="gaussian">
-                            <mean>0.0</mean>
-                            <stddev>1.7e-2</stddev>
-                            <bias_mean>0.1</bias_mean>
-                            <bias_stddev>0.001</bias_stddev>
-                        </noise>
-                    </z>
-                </linear_acceleration>
-            </imu>
-        </sensor>
-    </gazebo>
-    <!-- differential_drive_controller plugin -->
-    <gazebo>
-        <plugin name="differential_drive_controller" filename="libgazebo_ros_diff_drive.so">
-            <ros>
-                <namespace>/bot</namespace>
-                <!-- <argument>cmd_vel:=cmd_demo</argument>
-                <argument>odom:=odom_demo</argument> -->
-            </ros>
-            <robot_base_frame>base_link</robot_base_frame>
-            <update_rate>100</update_rate>
-            <left_joint>left_wheel_joint</left_joint>
-            <right_joint>right_wheel_joint</right_joint>
-            <wheel_separation>0.26</wheel_separation>
-            <wheel_diameter>0.2</wheel_diameter>
-            <publish_odom>true</publish_odom>
-            <publish_odom_tf>false</publish_odom_tf>
-            <publish_wheel_tf>true</publish_wheel_tf>
-            <odometry_frame>odom</odometry_frame>
-            <max_wheel_torque>10</max_wheel_torque>
-            <!-- Wheel acceleration, in rad/s^2, defaults to 0.0 rad/s^2 -->
-            <max_acceleration>1.0</max_acceleration>
-        </plugin>
-    </gazebo>
+<robot xmlns:xacro="http://www.ros.org/wiki/xacro" name="homeplater">
+    <xacro:include filename="$(find hpr_description)/urdf/hpr_core.urdf.xacro" />
 </robot>

Commit message: adapt physical properties

File: hpr_description/urdf/homeplater.urdf.xacro (robot description, xacro)
@@ -14,4 +14,5 @@
     <xacro:property name="base_width" value="0.16" />
     <xacro:property name="base_height" value="0.005" />
+    <xacro:property name="base_mass" value="0.2" />
     <!-- wheel properties -->
     <xacro:property name="wheel_xoffset" value="0.048" />
@@ -20,4 +21,5 @@
     <xacro:property name="wheel_radius" value="0.0325" />
     <xacro:property name="wheel_width" value="0.027" />
+    <xacro:property name="wheel_mass" value="0.032" />
     <!-- caster properties -->
     <xacro:property name="caster_xoffset" value="-0.044" />
@@ -25,4 +27,25 @@
     <xacro:property name="caster_radius" value="0.014" />
     <xacro:property name="caster_mass" value="0.1" />
+    <!-- inertial macro -->
+    <xacro:macro name="box_inertia" params="m d w h">
+        <inertial>
+            <origin xyz="0 0 0" rpy="${pi/2} 0 ${pi/2}" />
+            <mass value="${m}" />
+            <inertia ixx="${(m/12) * (h*h + w*w)}" ixy="0.0" ixz="0.0" iyy="${(m/12) * (d*d + h*h)}" iyz="0.0" izz="${(m/12) * (w*w + d*d)}" />
+        </inertial>
+    </xacro:macro>
+    <xacro:macro name="cylinder_inertia" params="m r h">
+        <inertial>
+            <origin xyz="0 0 0" rpy="${pi/2} 0 0" />
+            <mass value="${m}" />
+            <inertia ixx="${(m/12) * (3*r*r + h*h)}" ixy="0" ixz="0" iyy="${(m/12) * (3*r*r + h*h)}" iyz="0" izz="${(m/2) * (r*r)}" />
+        </inertial>
+    </xacro:macro>
+    <xacro:macro name="sphere_inertia" params="m r">
+        <inertial>
+            <mass value="${m}" />
+            <inertia ixx="${(2/5) * m * (r*r)}" ixy="0.0" ixz="0.0" iyy="${(2/5) * m * (r*r)}" iyz="0.0" izz="${(2/5) * m * (r*r)}" />
+        </inertial>
+    </xacro:macro>
     <!-- Wheel macro -->
     <xacro:macro name="wheel" params="prefix y_reflect">
@@ -40,4 +63,10 @@
                 <material name="black" />
             </visual>
+            <collision>
+                <geometry>
+                    <cylinder radius="${wheel_radius}" length="${wheel_width}" />
+                </geometry>
+            </collision>
+            <xacro:cylinder_inertia m="${wheel_mass}" r="${wheel_radius}" h="${wheel_width}" />
         </link>
     </xacro:macro>
@@ -50,4 +79,10 @@
             <material name="purple"/>
         </visual>
+        <collision>
+            <geometry>
+                <box size="${base_depth} ${base_width} ${base_height}"/>
+            </geometry>
+        </collision>
+        <xacro:box_inertia m="${base_mass}" d="${base_depth}" w="${base_width}" h="${base_height}" />
     </link>
     <joint name="caster_joint" type="fixed">
@@ -64,4 +99,10 @@
             <material name="gray" />
         </visual>
+        <collision>
+            <geometry>
+                <sphere radius="${caster_radius}" />
+            </geometry>
+        </collision>
+        <xacro:sphere_inertia m="${caster_mass}" r="${caster_radius}" />
     </link>
     <!-- LEFT AND RIGHT WHEEL -->

Commit message: add diif_drive plugin but not working

File: hpr_description/urdf/homeplater.urdf.xacro (robot description, xacro)
@@ -70,4 +70,7 @@
             <xacro:cylinder_inertia m="${wheel_mass}" r="${wheel_radius}" h="${wheel_width}" />
         </link>
+        <gazebo reference="${prefix}_link">
+            <material>Gazebo/Black</material>
+        </gazebo>
     </xacro:macro>
     <!-- BASE -->
@@ -86,4 +89,7 @@
         <xacro:box_inertia m="${base_mass}" d="${base_depth}" w="${base_width}" h="${base_height}" />
     </link>
+    <gazebo reference="base_link">
+        <material>Gazebo/Purple</material>
+    </gazebo>
     <joint name="caster_joint" type="fixed">
         <parent link="base_link" />
@@ -106,6 +112,31 @@
         <xacro:sphere_inertia m="${caster_mass}" r="${caster_radius}" />
     </link>
+    <gazebo reference="caster">
+        <material>Gazebo/Gray</material>
+    </gazebo>
     <!-- LEFT AND RIGHT WHEEL -->
     <xacro:wheel prefix="left_wheel" y_reflect="1" />
     <xacro:wheel prefix="right_wheel" y_reflect="-1" />
+    <gazebo>
+        <plugin name="differential_drive_controller" filename="libgazebo_ros_diff_drive.so">
+            <ros>
+                <namespace>/homeplater</namespace>
+                <!-- <argument>cmd_vel:=cmd_demo</argument>
+                <argument>odom:=odom_demo</argument> -->
+            </ros>
+            <robot_base_frame>base_link</robot_base_frame>
+            <update_rate>50</update_rate>
+            <left_joint>left_wheel_joint</left_joint>
+            <right_joint>right_wheel_joint</right_joint>
+            <wheel_separation>0.19</wheel_separation>
+            <wheel_diameter>0.065</wheel_diameter>
+            <publish_odom>true</publish_odom>
+            <publish_odom_tf>false</publish_odom_tf>
+            <publish_wheel_tf>true</publish_wheel_tf>
+            <odometry_frame>odom</odometry_frame>
+            <max_wheel_torque>20</max_wheel_torque>
+            <!-- Wheel acceleration, in rad/s^2, defaults to 0.0 rad/s^2 -->
+            <max_acceleration>1.0</max_acceleration>
+        </plugin>
+    </gazebo>
 </robot>

Commit message: fix dif_drive plugin

File: hpr_description/urdf/homeplater.urdf.xacro (robot description, xacro)
@@ -53,5 +53,5 @@
             <parent link="base_link" />
             <child link="${prefix}_link" />
-            <origin xyz="${wheel_xoffset} ${y_reflect*wheel_yoffset} ${wheel_zoffset}" rpy="${pi/2} 0 0" />
+            <origin xyz="${wheel_xoffset} ${y_reflect*wheel_yoffset} ${wheel_zoffset}" rpy="${-pi/2} 0 0" />
             <axis xyz="0 0 1" />
         </joint>
@@ -113,4 +113,6 @@
     </link>
     <gazebo reference="caster">
+        <mu1>0.0001</mu1>
+        <mu2>0.0001</mu2>
         <material>Gazebo/Gray</material>
     </gazebo>
@@ -132,5 +134,5 @@
             <wheel_diameter>0.065</wheel_diameter>
             <publish_odom>true</publish_odom>
-            <publish_odom_tf>false</publish_odom_tf>
+            <publish_odom_tf>true</publish_odom_tf>
             <publish_wheel_tf>true</publish_wheel_tf>
             <odometry_frame>odom</odometry_frame>

Commit message: update urdf

File: hpr_description/urdf/homeplater.urdf.xacro (robot description, xacro)
@@ -22,7 +22,5 @@
     <!-- caster properties -->
     <xacro:property name="caster_xoffset" value="-0.044" />
-    <!-- <xacro:property name="caster_zoffset" value="-0.0315" /> -->
     <xacro:property name="caster_radius" value="0.014" />
-    <xacro:property name="caster_mass" value="0.1" />
     <!-- Wheel macro -->
     <xacro:macro name="wheel" params="prefix y_reflect">
@@ -30,5 +28,5 @@
             <parent link="base_link" />
             <child link="${prefix}_link" />
-            <origin xyz="${wheel_xoffset} ${y_reflect*wheel_yoffset} ${wheel_zoffset}" rpy="${pi/2} 0 0" />
+            <origin xyz="${wheel_xoffset} ${y_reflect*wheel_yoffset} ${wheel_zoffset}" rpy="${-pi/2} 0 0" />
             <axis xyz="0 0 1" />
         </joint>

Commit message: update wheel joint rpy

File: hpr_description/urdf/homeplater.urdf.xacro (robot description, xacro)
@@ -53,5 +53,5 @@
             <parent link="base_link" />
             <child link="${prefix}_link" />
-            <origin xyz="${wheel_xoffset} ${y_reflect*wheel_yoffset} ${wheel_zoffset}" rpy="${pi/2} 0 0" />
+            <origin xyz="${wheel_xoffset} ${y_reflect*wheel_yoffset} ${wheel_zoffset}" rpy="${-pi/2} 0 0" />
             <axis xyz="0 0 1" />
         </joint>

Commit message: update wheel joint rpy

File: hpr_description/urdf/homeplater.urdf.xacro (robot description, xacro)
@@ -24,5 +24,4 @@
     <!-- caster properties -->
     <xacro:property name="caster_xoffset" value="-0.044" />
-    <!-- <xacro:property name="caster_zoffset" value="-0.0315" /> -->
     <xacro:property name="caster_radius" value="0.014" />
     <xacro:property name="caster_mass" value="0.1" />
@@ -53,5 +52,5 @@
             <parent link="base_link" />
             <child link="${prefix}_link" />
-            <origin xyz="${wheel_xoffset} ${y_reflect*wheel_yoffset} ${wheel_zoffset}" rpy="${pi/2} 0 0" />
+            <origin xyz="${wheel_xoffset} ${y_reflect*wheel_yoffset} ${wheel_zoffset}" rpy="${-pi/2} 0 0" />
             <axis xyz="0 0 1" />
         </joint>
