Commit message: update diffdrive plugin

File: hpr_description/urdf/homeplater.urdf.xacro (robot description, xacro)
@@ -24,5 +24,4 @@
     <!-- caster properties -->
     <xacro:property name="caster_xoffset" value="-0.044" />
-    <!-- <xacro:property name="caster_zoffset" value="-0.0315" /> -->
     <xacro:property name="caster_radius" value="0.014" />
     <xacro:property name="caster_mass" value="0.1" />
@@ -127,17 +126,21 @@
                 <argument>odom:=odom_demo</argument> -->
             </ros>
-            <robot_base_frame>base_link</robot_base_frame>
-            <update_rate>50</update_rate>
+            <!-- wheels -->
             <left_joint>left_wheel_joint</left_joint>
             <right_joint>right_wheel_joint</right_joint>
+            <!-- kinematics -->
             <wheel_separation>0.19</wheel_separation>
             <wheel_diameter>0.065</wheel_diameter>
+            <!-- tfs -->
             <publish_odom>true</publish_odom>
             <publish_odom_tf>true</publish_odom_tf>
             <publish_wheel_tf>true</publish_wheel_tf>
             <odometry_frame>odom</odometry_frame>
+            <!-- limits -->
             <max_wheel_torque>20</max_wheel_torque>
-            <!-- Wheel acceleration, in rad/s^2, defaults to 0.0 rad/s^2 -->
             <max_acceleration>1.0</max_acceleration>
+            <!-- miscs -->
+            <robot_base_frame>base_link</robot_base_frame>
+            <update_rate>50</update_rate>
         </plugin>
     </gazebo>

Commit message: update urdf with lidar

File: hpr_description/urdf/homeplater.urdf.xacro (robot description, xacro)
@@ -25,5 +25,10 @@
     <xacro:property name="caster_xoffset" value="-0.044" />
     <xacro:property name="caster_radius" value="0.014" />
-    <xacro:property name="caster_mass" value="0.1" />
+    <xacro:property name="caster_mass" value="0.05" />
+    <!-- lidar properties -->
+    <xacro:property name="lidar_radius" value="0.035" />
+    <xacro:property name="lidar_height" value="0.02" />
+    <xacro:property name="lidar_zoff" value="0.08" />
+    <xacro:property name="lidar_mass" value="0.17" />
     <!-- inertial macro -->
     <xacro:macro name="box_inertia" params="m d w h">
@@ -145,3 +150,59 @@
         </plugin>
     </gazebo>
+    <!-- LIDAR -->
+    <joint name="lidar_joint" type="fixed">
+        <parent link="base_link" />
+        <child link="lidar" />
+        <origin xyz="0 0 ${(base_height+lidar_height)/2+lidar_zoff}" />
+    </joint>
+    <link name="lidar">
+        <visual>
+            <geometry>
+                <cylinder radius="${lidar_radius}" length="${lidar_height}" />
+            </geometry>
+            <material name="black" />
+        </visual>
+        <collision>
+            <origin xyz="0 0 0" rpy="0 0 0" />
+            <geometry>
+                <cylinder radius="${lidar_radius}" length="${lidar_height}" />
+            </geometry>
+        </collision>
+        <xacro:cylinder_inertia m="${lidar_mass}" r="${lidar_radius}" h="${lidar_height}" />
+    </link>
+    <gazebo reference="lidar">
+        <material>Gazebo/Black</material>
+        <sensor name="lidar" type="ray">
+            <always_on>true</always_on>
+            <visualize>true</visualize>
+            <update_rate>5</update_rate>
+            <ray>
+                <scan>
+                    <horizontal>
+                        <samples>360</samples>
+                        <resolution>1.000000</resolution>
+                        <min_angle>0.000000</min_angle>
+                        <max_angle>6.280000</max_angle>
+                    </horizontal>
+                </scan>
+                <range>
+                    <min>0.120000</min>
+                    <max>6</max>
+                    <resolution>0.015000</resolution>
+                </range>
+                <noise>
+                    <type>gaussian</type>
+                    <mean>0.0</mean>
+                    <stddev>0.01</stddev>
+                </noise>
+            </ray>
+            <plugin name="scan" filename="libgazebo_ros_ray_sensor.so">
+                <ros>
+                    <remapping>~/out:=scan</remapping>
+                </ros>
+                <output_type>sensor_msgs/LaserScan</output_type>
+                <frame_name>lidar</frame_name>
+            </plugin>
+        </sensor>
+    </gazebo>
 </robot>

Commit message: init branch

File: hpr_description/urdf/homeplater.urdf.xacro (robot description, xacro)
@@ -1,208 +1,4 @@
 <?xml version="1.0"?>
 <robot xmlns:xacro="http://www.ros.org/wiki/xacro" name="homeplater">
-    <material name="black">
-        <color rgba="0 0 0 1"/>
-    </material>
-    <material name="purple">
-        <color rgba="0.3098 0.1765 0.4980 1" />
-    </material>
-    <material name="gray">
-        <color rgba="0.5 0.5 0.5 1" />
-    </material>
-    <!-- base properties -->
-    <xacro:property name="base_depth" value="0.16" />
-    <xacro:property name="base_width" value="0.16" />
-    <xacro:property name="base_height" value="0.005" />
-    <xacro:property name="base_mass" value="0.2" />
-    <!-- wheel properties -->
-    <xacro:property name="wheel_xoffset" value="0.048" />
-    <xacro:property name="wheel_yoffset" value="0.095" />
-    <xacro:property name="wheel_zoffset" value="-0.013" />
-    <xacro:property name="wheel_radius" value="0.0325" />
-    <xacro:property name="wheel_width" value="0.027" />
-    <xacro:property name="wheel_mass" value="0.032" />
-    <!-- caster properties -->
-    <xacro:property name="caster_xoffset" value="-0.044" />
-    <xacro:property name="caster_radius" value="0.014" />
-    <xacro:property name="caster_mass" value="0.05" />
-    <!-- lidar properties -->
-    <xacro:property name="lidar_radius" value="0.035" />
-    <xacro:property name="lidar_height" value="0.02" />
-    <xacro:property name="lidar_zoff" value="0.08" />
-    <xacro:property name="lidar_mass" value="0.17" />
-    <!-- inertial macro -->
-    <xacro:macro name="box_inertia" params="m d w h">
-        <inertial>
-            <origin xyz="0 0 0" rpy="${pi/2} 0 ${pi/2}" />
-            <mass value="${m}" />
-            <inertia ixx="${(m/12) * (h*h + w*w)}" ixy="0.0" ixz="0.0" iyy="${(m/12) * (d*d + h*h)}" iyz="0.0" izz="${(m/12) * (w*w + d*d)}" />
-        </inertial>
-    </xacro:macro>
-    <xacro:macro name="cylinder_inertia" params="m r h">
-        <inertial>
-            <origin xyz="0 0 0" rpy="${pi/2} 0 0" />
-            <mass value="${m}" />
-            <inertia ixx="${(m/12) * (3*r*r + h*h)}" ixy="0" ixz="0" iyy="${(m/12) * (3*r*r + h*h)}" iyz="0" izz="${(m/2) * (r*r)}" />
-        </inertial>
-    </xacro:macro>
-    <xacro:macro name="sphere_inertia" params="m r">
-        <inertial>
-            <mass value="${m}" />
-            <inertia ixx="${(2/5) * m * (r*r)}" ixy="0.0" ixz="0.0" iyy="${(2/5) * m * (r*r)}" iyz="0.0" izz="${(2/5) * m * (r*r)}" />
-        </inertial>
-    </xacro:macro>
-    <!-- Wheel macro -->
-    <xacro:macro name="wheel" params="prefix y_reflect">
-        <joint name="${prefix}_joint" type="continuous">
-            <parent link="base_link" />
-            <child link="${prefix}_link" />
-            <origin xyz="${wheel_xoffset} ${y_reflect*wheel_yoffset} ${wheel_zoffset}" rpy="${-pi/2} 0 0" />
-            <axis xyz="0 0 1" />
-        </joint>
-        <link name="${prefix}_link">
-            <visual>
-                <geometry>
-                    <cylinder radius="${wheel_radius}" length="${wheel_width}" />
-                </geometry>
-                <material name="black" />
-            </visual>
-            <collision>
-                <geometry>
-                    <cylinder radius="${wheel_radius}" length="${wheel_width}" />
-                </geometry>
-            </collision>
-            <xacro:cylinder_inertia m="${wheel_mass}" r="${wheel_radius}" h="${wheel_width}" />
-        </link>
-        <gazebo reference="${prefix}_link">
-            <material>Gazebo/Black</material>
-        </gazebo>
-    </xacro:macro>
-    <!-- BASE -->
-    <link name="base_link">
-        <visual>
-            <geometry>
-                <box size="${base_depth} ${base_width} ${base_height}"/>
-            </geometry>
-            <material name="purple"/>
-        </visual>
-        <collision>
-            <geometry>
-                <box size="${base_depth} ${base_width} ${base_height}"/>
-            </geometry>
-        </collision>
-        <xacro:box_inertia m="${base_mass}" d="${base_depth}" w="${base_width}" h="${base_height}" />
-    </link>
-    <gazebo reference="base_link">
-        <material>Gazebo/Purple</material>
-    </gazebo>
-    <joint name="caster_joint" type="fixed">
-        <parent link="base_link" />
-        <child link="caster" />
-        <origin xyz="${caster_xoffset} 0.0 ${caster_radius-wheel_radius+wheel_zoffset}" />
-    </joint>
-    <!-- CASTER WHEEL -->
-    <link name="caster">
-        <visual>
-            <geometry>
-                <sphere radius="${caster_radius}" />
-            </geometry>
-            <material name="gray" />
-        </visual>
-        <collision>
-            <geometry>
-                <sphere radius="${caster_radius}" />
-            </geometry>
-        </collision>
-        <xacro:sphere_inertia m="${caster_mass}" r="${caster_radius}" />
-    </link>
-    <gazebo reference="caster">
-        <mu1>0.0001</mu1>
-        <mu2>0.0001</mu2>
-        <material>Gazebo/Gray</material>
-    </gazebo>
-    <!-- LEFT AND RIGHT WHEEL -->
-    <xacro:wheel prefix="left_wheel" y_reflect="1" />
-    <xacro:wheel prefix="right_wheel" y_reflect="-1" />
-    <gazebo>
-        <plugin name="differential_drive_controller" filename="libgazebo_ros_diff_drive.so">
-            <ros>
-                <namespace>/homeplater</namespace>
-                <!-- <argument>cmd_vel:=cmd_demo</argument>
-                <argument>odom:=odom_demo</argument> -->
-            </ros>
-            <!-- wheels -->
-            <left_joint>left_wheel_joint</left_joint>
-            <right_joint>right_wheel_joint</right_joint>
-            <!-- kinematics -->
-            <wheel_separation>0.19</wheel_separation>
-            <wheel_diameter>0.065</wheel_diameter>
-            <!-- tfs -->
-            <publish_odom>true</publish_odom>
-            <publish_odom_tf>true</publish_odom_tf>
-            <publish_wheel_tf>true</publish_wheel_tf>
-            <odometry_frame>odom</odometry_frame>
-            <!-- limits -->
-            <max_wheel_torque>20</max_wheel_torque>
-            <max_acceleration>1.0</max_acceleration>
-            <!-- miscs -->
-            <robot_base_frame>base_link</robot_base_frame>
-            <update_rate>50</update_rate>
-        </plugin>
-    </gazebo>
-    <!-- LIDAR -->
-    <joint name="lidar_joint" type="fixed">
-        <parent link="base_link" />
-        <child link="lidar" />
-        <origin xyz="0 0 ${(base_height+lidar_height)/2+lidar_zoff}" />
-    </joint>
-    <link name="lidar">
-        <visual>
-            <geometry>
-                <cylinder radius="${lidar_radius}" length="${lidar_height}" />
-            </geometry>
-            <material name="black" />
-        </visual>
-        <collision>
-            <origin xyz="0 0 0" rpy="0 0 0" />
-            <geometry>
-                <cylinder radius="${lidar_radius}" length="${lidar_height}" />
-            </geometry>
-        </collision>
-        <xacro:cylinder_inertia m="${lidar_mass}" r="${lidar_radius}" h="${lidar_height}" />
-    </link>
-    <gazebo reference="lidar">
-        <material>Gazebo/Black</material>
-        <sensor name="lidar" type="ray">
-            <always_on>true</always_on>
-            <visualize>true</visualize>
-            <update_rate>5</update_rate>
-            <ray>
-                <scan>
-                    <horizontal>
-                        <samples>360</samples>
-                        <resolution>1.000000</resolution>
-                        <min_angle>0.000000</min_angle>
-                        <max_angle>6.280000</max_angle>
-                    </horizontal>
-                </scan>
-                <range>
-                    <min>0.120000</min>
-                    <max>6</max>
-                    <resolution>0.015000</resolution>
-                </range>
-                <noise>
-                    <type>gaussian</type>
-                    <mean>0.0</mean>
-                    <stddev>0.01</stddev>
-                </noise>
-            </ray>
-            <plugin name="scan" filename="libgazebo_ros_ray_sensor.so">
-                <ros>
-                    <remapping>~/out:=scan</remapping>
-                </ros>
-                <output_type>sensor_msgs/LaserScan</output_type>
-                <frame_name>lidar</frame_name>
-            </plugin>
-        </sensor>
-    </gazebo>
+    <xacro:include filename="$(find hpr_description)/urdf/hpr_core.urdf.xacro" />
 </robot>

Commit message: add libgazebo_diff_drive_plugin

File: hpr_description/urdf/homeplater.urdf.xacro (robot description, xacro)
@@ -1,4 +1,6 @@
 <?xml version="1.0"?>
 <robot xmlns:xacro="http://www.ros.org/wiki/xacro" name="homeplater">
-    <xacro:include filename="$(find hpr_description)/urdf/hpr_core.urdf.xacro" />
+    <!-- <xacro:include filename="$(find hpr_description)/urdf/hpr_core.urdf.xacro" /> -->
+    <xacro:include filename="hpr_core.urdf.xacro" />
+    <xacro:include filename="gazebo_ros_diff_drive.xacro" />
 </robot>

File: hpr_description/urdf/hpr_core.urdf.xacro (robot description, xacro)
@@ -1,6 +1,8 @@
 <?xml version="1.0"?>
 <robot xmlns:xacro="http://www.ros.org/wiki/xacro" >
-    <xacro:include filename="$(find hpr_description)/urdf/materials.xacro" />
-    <xacro:include filename="$(find hpr_description)/urdf/inertia.xacro" />
+    <!-- <xacro:include filename="$(find hpr_description)/urdf/materials.xacro" />
+    <xacro:include filename="$(find hpr_description)/urdf/inertia.xacro" /> -->
+    <xacro:include filename="materials.xacro" />
+    <xacro:include filename="inertia.xacro" />
     <!-- base properties -->
     <xacro:property name="chassis_xoffset" value="-0.048" />
@@ -77,5 +79,5 @@
     </gazebo>
     <!-- CASTER WHEEL -->
-    <!-- <joint name="caster_joint" type="fixed">
+    <joint name="caster_joint" type="fixed">
         <parent link="base_link" />
         <child link="caster_link" />
@@ -100,7 +102,7 @@
         <mu2>0.00000001</mu2>
         <material>Gazebo/Gray</material>
-    </gazebo> -->
+    </gazebo>
     <!-- LEFT AND RIGHT WHEEL -->
-    <!-- <xacro:wheel prefix="left_wheel" y_reflect="1" />
-    <xacro:wheel prefix="right_wheel" y_reflect="-1" /> -->
+    <xacro:wheel prefix="left_wheel" y_reflect="1" />
+    <xacro:wheel prefix="right_wheel" y_reflect="-1" />
 </robot>

Commit message: update inertial macro

File: hpr_description/urdf/homeplater.urdf.xacro (robot description, xacro)
@@ -30,5 +30,4 @@
     <xacro:macro name="box_inertia" params="m d w h">
         <inertial>
-            <origin xyz="0 0 0" rpy="${pi/2} 0 ${pi/2}" />
             <mass value="${m}" />
             <inertia ixx="${(m/12) * (h*h + w*w)}" ixy="0.0" ixz="0.0" iyy="${(m/12) * (d*d + h*h)}" iyz="0.0" izz="${(m/12) * (w*w + d*d)}" />
@@ -37,5 +36,4 @@
     <xacro:macro name="cylinder_inertia" params="m r h">
         <inertial>
-            <origin xyz="0 0 0" rpy="${pi/2} 0 0" />
             <mass value="${m}" />
             <inertia ixx="${(m/12) * (3*r*r + h*h)}" ixy="0" ixz="0" iyy="${(m/12) * (3*r*r + h*h)}" iyz="0" izz="${(m/2) * (r*r)}" />

Commit message: update inertial macro

File: hpr_description/urdf/homeplater.urdf.xacro (robot description, xacro)
@@ -29,5 +29,4 @@
     <xacro:macro name="box_inertia" params="m d w h">
         <inertial>
-            <origin xyz="0 0 0" rpy="${pi/2} 0 ${pi/2}" />
             <mass value="${m}" />
             <inertia ixx="${(m/12) * (h*h + w*w)}" ixy="0.0" ixz="0.0" iyy="${(m/12) * (d*d + h*h)}" iyz="0.0" izz="${(m/12) * (w*w + d*d)}" />
@@ -36,5 +35,4 @@
     <xacro:macro name="cylinder_inertia" params="m r h">
         <inertial>
-            <origin xyz="0 0 0" rpy="${pi/2} 0 0" />
             <mass value="${m}" />
             <inertia ixx="${(m/12) * (3*r*r + h*h)}" ixy="0" ixz="0" iyy="${(m/12) * (3*r*r + h*h)}" iyz="0" izz="${(m/2) * (r*r)}" />

Commit message: update inertial macro

File: hpr_description/urdf/homeplater.urdf.xacro (robot description, xacro)
@@ -34,5 +34,4 @@
     <xacro:macro name="box_inertia" params="m d w h">
         <inertial>
-            <origin xyz="0 0 0" rpy="${pi/2} 0 ${pi/2}" />
             <mass value="${m}" />
             <inertia ixx="${(m/12) * (h*h + w*w)}" ixy="0.0" ixz="0.0" iyy="${(m/12) * (d*d + h*h)}" iyz="0.0" izz="${(m/12) * (w*w + d*d)}" />
@@ -41,5 +40,4 @@
     <xacro:macro name="cylinder_inertia" params="m r h">
         <inertial>
-            <origin xyz="0 0 0" rpy="${pi/2} 0 0" />
             <mass value="${m}" />
             <inertia ixx="${(m/12) * (3*r*r + h*h)}" ixy="0" ixz="0" iyy="${(m/12) * (3*r*r + h*h)}" iyz="0" izz="${(m/2) * (r*r)}" />
