Commit message: sync with branch 6

File: hpr_description/urdf/homeplater.urdf.xacro (robot description, xacro)
@@ -1,4 +1,8 @@
 <?xml version="1.0"?>
 <robot xmlns:xacro="http://www.ros.org/wiki/xacro" name="homeplater">
-    <xacro:include filename="$(find hpr_description)/urdf/hpr_core.urdf.xacro" />
+    <!-- <xacro:include filename="$(find hpr_description)/urdf/hpr_core.urdf.xacro" /> -->
+    <xacro:include filename="hpr_core.urdf.xacro" />
+    <xacro:include filename="lidar.urdf.xacro" />
+    <xacro:include filename="gazebo_ros_diff_drive.xacro" />
+    <xacro:include filename="gazebo_ros_ray.xacro" />
 </robot>

File: hpr_description/urdf/hpr_core.urdf.xacro (robot description, xacro)
@@ -1,23 +1,29 @@
 <?xml version="1.0"?>
 <robot xmlns:xacro="http://www.ros.org/wiki/xacro" >
-    <!-- Import colors -->
-    <xacro:include filename="$(find hpr_description)/urdf/materials.xacro" />
-    <!-- Import inertia -->
-    <xacro:include filename="$(find hpr_description)/urdf/inertia.xacro" />
-    <!-- Define properties -->
+    <!-- <xacro:include filename="$(find hpr_description)/urdf/materials.xacro" />
+    <xacro:include filename="$(find hpr_description)/urdf/inertia.xacro" /> -->
+    <xacro:include filename="materials.xacro" />
+    <xacro:include filename="inertia.xacro" />
     <!-- base properties -->
-    <xacro:property name="base_width" value="0.16" />
-    <xacro:property name="base_depth" value="0.16" />
-    <xacro:property name="base_height" value="0.005" />
-    <xacro:property name="base_mass" value="1.0" />
+    <xacro:property name="chassis_xoffset" value="-0.048" />
+    <xacro:property name="chassis_zoffset" value="0.013" />
+    <xacro:property name="chassis_depth" value="0.16" />
+    <xacro:property name="chassis_width" value="0.16" />
+    <xacro:property name="chassis_height" value="0.005" />
+    <xacro:property name="chassis_mass" value="0.2" />
     <!-- wheel properties -->
-    <xacro:property name="wheel_offset" value="0.095" />
+    <xacro:property name="wheel_yoffset" value="0.095" />
     <xacro:property name="wheel_radius" value="0.0325" />
     <xacro:property name="wheel_width" value="0.027" />
     <xacro:property name="wheel_mass" value="0.032" />
     <!-- caster properties -->
-    <xacro:property name="caster_xoff" value="-0.092" />
+    <xacro:property name="caster_xoffset" value="-0.092" />
     <xacro:property name="caster_radius" value="0.014" />
-    <xacro:property name="caster_mass" value="0.1" />
+    <xacro:property name="caster_mass" value="0.05" />
+    <!-- lidar properties -->
+    <xacro:property name="lidar_radius" value="0.035" />
+    <xacro:property name="lidar_height" value="0.02" />
+    <xacro:property name="lidar_zoff" value="0.08" />
+    <xacro:property name="lidar_mass" value="0.17" />
     <!-- Wheel macro -->
     <xacro:macro name="wheel" params="prefix y_reflect">
@@ -25,5 +31,5 @@
             <parent link="base_link" />
             <child link="${prefix}_link" />
-            <origin xyz="0 ${y_reflect*wheel_offset} 0" rpy="${pi/2} 0 0" />
+            <origin xyz="0 ${y_reflect*wheel_yoffset} 0" rpy="${-pi/2} 0 0" />
             <axis xyz="0 0 1" />
         </joint>
@@ -42,18 +48,21 @@
             <xacro:cylinder_inertia m="${wheel_mass}" r="${wheel_radius}" h="${wheel_width}" />
         </link>
+        <gazebo reference="${prefix}_link">
+            <material>Gazebo/Black</material>
+        </gazebo>
     </xacro:macro>
-    <!-- CENTER OF WHEEL BASE -->
+    <!-- DUMMY BASE -->
     <link name="base_link">
     </link>
     <!-- CHASSIS -->
     <joint name="chassis_joint" type="fixed">
-        <parent link="base_link"/>
-        <child link="chassis"/>
-        <origin xyz="-0.048 0 0.013"/>
+        <parent link="base_link" />
+        <child link="chassis_link" />
+        <origin xyz="${chassis_xoffset} 0 ${chassis_zoffset}" />
     </joint>
-    <link name="chassis">
+    <link name="chassis_link">
         <visual>
             <geometry>
-                <box size="${base_depth} ${base_width} ${base_height}"/>
+                <box size="${chassis_depth} ${chassis_width} ${chassis_height}"/>
             </geometry>
             <material name="purple"/>
@@ -61,24 +70,19 @@
         <collision>
             <geometry>
-                <box size="${base_depth} ${base_width} ${base_height}"/>
+                <box size="${chassis_depth} ${chassis_width} ${chassis_height}"/>
             </geometry>
-            <material name="purple"/>
         </collision>
-        <xacro:box_inertia m="${base_mass}" d="${base_depth}" w="${base_width}" h="${base_height}" />
+        <xacro:box_inertia m="${chassis_mass}" x="${chassis_depth}" y="${chassis_width}" z="${chassis_height}" />
     </link>
-    <gazebo reference="chassis">
+    <gazebo reference="chassis_link">
         <material>Gazebo/Purple</material>
     </gazebo>
-    <!-- LEFT WHEEL -->
-    <xacro:wheel prefix="left_wheel" y_reflect="1" />
-    <!-- RIGHT WHEEL -->
-    <xacro:wheel prefix="right_wheel" y_reflect="-1" />
-    <!-- CASTER BALL -->
+    <!-- CASTER WHEEL -->
     <joint name="caster_joint" type="fixed">
         <parent link="base_link" />
-        <child link="caster" />
-        <origin xyz="${caster_xoff} 0.0 ${caster_radius-wheel_radius}" />
+        <child link="caster_link" />
+        <origin xyz="${caster_xoffset} 0.0 ${caster_radius-wheel_radius}" />
     </joint>
-    <link name="caster">
+    <link name="caster_link">
         <visual>
             <geometry>
@@ -94,25 +98,11 @@
         <xacro:sphere_inertia m="${caster_mass}" r="${caster_radius}" />
     </link>
-    <gazebo>
-        <plugin name="differential_drive_controller" filename="libgazebo_ros_diff_drive.so">
-            <ros>
-                <namespace>/homeplater</namespace>
-                <!-- <argument>cmd_vel:=cmd_demo</argument>
-                <argument>odom:=odom_demo</argument> -->
-            </ros>
-            <robot_base_frame>base_link</robot_base_frame>
-            <update_rate>100</update_rate>
-            <left_joint>left_wheel_joint</left_joint>
-            <right_joint>right_wheel_joint</right_joint>
-            <wheel_separation>0.19</wheel_separation>
-            <wheel_diameter>0.065</wheel_diameter>
-            <publish_odom>true</publish_odom>
-            <publish_odom_tf>false</publish_odom_tf>
-            <publish_wheel_tf>true</publish_wheel_tf>
-            <odometry_frame>odom</odometry_frame>
-            <max_wheel_torque>10</max_wheel_torque>
-            <!-- Wheel acceleration, in rad/s^2, defaults to 0.0 rad/s^2 -->
-            <max_acceleration>1.0</max_acceleration>
-        </plugin>
+    <gazebo reference="caster_link">
+        <mu1>0.00000001</mu1>
+        <mu2>0.00000001</mu2>
+        <material>Gazebo/Gray</material>
     </gazebo>
+    <!-- LEFT AND RIGHT WHEEL -->
+    <xacro:wheel prefix="left_wheel" y_reflect="1" />
+    <xacro:wheel prefix="right_wheel" y_reflect="-1" />
 </robot>

File: hpr_description/urdf/inertia.xacro (robot description, xacro)
@@ -1,14 +1,13 @@
 <?xml version="1.0"?>
 <robot xmlns:xacro="http://www.ros.org/wiki/xacro" >
-    <xacro:macro name="box_inertia" params="m d w h">
+    <!-- inertial macro -->
+    <xacro:macro name="box_inertia" params="m x y z">
         <inertial>
-            <origin xyz="0 0 0" rpy="${pi/2} 0 ${pi/2}" />
             <mass value="${m}" />
-            <inertia ixx="${(m/12) * (h*h + w*w)}" ixy="0.0" ixz="0.0" iyy="${(m/12) * (d*d + h*h)}" iyz="0.0" izz="${(m/12) * (w*w + d*d)}" />
+            <inertia ixx="${(m/12) * (y*y + z*z)}" ixy="0.0" ixz="0.0" iyy="${(m/12) * (z*z + x*x)}" iyz="0.0" izz="${(m/12) * (x*x + y*y)}" />
         </inertial>
     </xacro:macro>
     <xacro:macro name="cylinder_inertia" params="m r h">
         <inertial>
-            <origin xyz="0 0 0" rpy="${pi/2} 0 0" />
             <mass value="${m}" />
             <inertia ixx="${(m/12) * (3*r*r + h*h)}" ixy="0" ixz="0" iyy="${(m/12) * (3*r*r + h*h)}" iyz="0" izz="${(m/2) * (r*r)}" />

Commit message: minor urdf fix

File: hpr_description/urdf/homeplater.urdf.xacro (robot description, xacro)
@@ -162,5 +162,4 @@
         </visual>
         <collision>
-            <origin xyz="0 0 0" rpy="0 0 0" />
             <geometry>
                 <cylinder radius="${lidar_radius}" length="${lidar_height}" />
