Commit message: fix dropping message: lidar

File: hpr_description/urdf/gazebo_ros_ray.xacro (robot description, xacro)
@@ -6,5 +6,5 @@
             <always_on>true</always_on>
             <visualize>true</visualize>
-            <update_rate>5</update_rate>
+            <update_rate>10</update_rate>
             <ray>
                 <scan>
@@ -32,5 +32,5 @@
                 </ros>
                 <output_type>sensor_msgs/LaserScan</output_type>
-                <frame_name>lidar</frame_name>
+                <!-- <frame_name>lidar</frame_name> -->
             </plugin>
         </sensor>

File: hpr_description/urdf/lidar.urdf.xacro (robot description, xacro)
@@ -21,5 +21,4 @@
         </visual>
         <collision>
-            <origin xyz="0 0 0" rpy="0 0 0" />
             <geometry>
                 <cylinder radius="${lidar_radius}" length="${lidar_height}" />
