Commit message: update model description with gazebo tags

File: hpr_description/urdf/hpr_core.urdf.xacro (robot description, xacro)
@@ -67,4 +67,7 @@
         <xacro:box_inertia m="${base_mass}" d="${base_depth}" w="${base_width}" h="${base_height}" />
     </link>
+    <gazebo reference="chassis">
+        <material>Gazebo/Purple</material>
+    </gazebo>
     <!-- LEFT WHEEL -->
     <xacro:wheel prefix="left_wheel" y_reflect="1" />
@@ -91,3 +94,25 @@
         <xacro:sphere_inertia m="${caster_mass}" r="${caster_radius}" />
     </link>
+    <gazebo>
+        <plugin name="differential_drive_controller" filename="libgazebo_ros_diff_drive.so">
+            <ros>
+                <namespace>/homeplater</namespace>
+                <!-- <argument>cmd_vel:=cmd_demo</argument>
+                <argument>odom:=odom_demo</argument> -->
+            </ros>
+            <robot_base_frame>base_link</robot_base_frame>
+            <update_rate>100</update_rate>
+            <left_joint>left_wheel_joint</left_joint>
+            <right_joint>right_wheel_joint</right_joint>
+            <wheel_separation>0.19</wheel_separation>
+            <wheel_diameter>0.065</wheel_diameter>
+            <publish_odom>true</publish_odom>
+            <publish_odom_tf>false</publish_odom_tf>
+            <publish_wheel_tf>true</publish_wheel_tf>
+            <odometry_frame>odom</odometry_frame>
+            <max_wheel_torque>10</max_wheel_torque>
+            <!-- Wheel acceleration, in rad/s^2, defaults to 0.0 rad/s^2 -->
+            <max_acceleration>1.0</max_acceleration>
+        </plugin>
+    </gazebo>
 </robot>

Commit message: separate materials and inertia

File: hpr_description/urdf/hpr_core.urdf.xacro (robot description, xacro)
@@ -1,13 +1,6 @@
 <?xml version="1.0"?>
 <robot xmlns:xacro="http://www.ros.org/wiki/xacro" >
-    <material name="black">
-        <color rgba="0 0 0 1"/>
-    </material>
-    <material name="purple">
-        <color rgba="0.3098 0.1765 0.4980 1" />
-    </material>
-    <material name="gray">
-        <color rgba="0.5 0.5 0.5 1" />
-    </material>
+    <xacro:include filename="$(find hpr_description)/urdf/materials.xacro" />
+    <xacro:include filename="$(find hpr_description)/urdf/inertia.xacro" />
     <!-- base properties -->
     <xacro:property name="base_depth" value="0.16" />
@@ -31,25 +24,4 @@
     <xacro:property name="lidar_zoff" value="0.08" />
     <xacro:property name="lidar_mass" value="0.17" />
-    <!-- inertial macro -->
-    <xacro:macro name="box_inertia" params="m d w h">
-        <inertial>
-            <origin xyz="0 0 0" rpy="${pi/2} 0 ${pi/2}" />
-            <mass value="${m}" />
-            <inertia ixx="${(m/12) * (h*h + w*w)}" ixy="0.0" ixz="0.0" iyy="${(m/12) * (d*d + h*h)}" iyz="0.0" izz="${(m/12) * (w*w + d*d)}" />
-        </inertial>
-    </xacro:macro>
-    <xacro:macro name="cylinder_inertia" params="m r h">
-        <inertial>
-            <origin xyz="0 0 0" rpy="${pi/2} 0 0" />
-            <mass value="${m}" />
-            <inertia ixx="${(m/12) * (3*r*r + h*h)}" ixy="0" ixz="0" iyy="${(m/12) * (3*r*r + h*h)}" iyz="0" izz="${(m/2) * (r*r)}" />
-        </inertial>
-    </xacro:macro>
-    <xacro:macro name="sphere_inertia" params="m r">
-        <inertial>
-            <mass value="${m}" />
-            <inertia ixx="${(2/5) * m * (r*r)}" ixy="0.0" ixz="0.0" iyy="${(2/5) * m * (r*r)}" iyz="0.0" izz="${(2/5) * m * (r*r)}" />
-        </inertial>
-    </xacro:macro>
     <!-- Wheel macro -->
     <xacro:macro name="wheel" params="prefix y_reflect">
@@ -91,5 +63,5 @@
             </geometry>
         </collision>
-        <xacro:box_inertia m="${base_mass}" d="${base_depth}" w="${base_width}" h="${base_height}" />
+        <xacro:box_inertia m="${base_mass}" x="${base_depth}" y="${base_width}" z="${base_height}" />
     </link>
     <gazebo reference="base_link">

Commit message: urdf start from dummy base_link

File: hpr_description/urdf/hpr_core.urdf.xacro (robot description, xacro)
@@ -4,17 +4,17 @@
     <xacro:include filename="$(find hpr_description)/urdf/inertia.xacro" />
     <!-- base properties -->
-    <xacro:property name="base_depth" value="0.16" />
-    <xacro:property name="base_width" value="0.16" />
-    <xacro:property name="base_height" value="0.005" />
-    <xacro:property name="base_mass" value="0.2" />
+    <xacro:property name="chassis_xoffset" value="-0.048" />
+    <xacro:property name="chassis_zoffset" value="0.013" />
+    <xacro:property name="chassis_depth" value="0.16" />
+    <xacro:property name="chassis_width" value="0.16" />
+    <xacro:property name="chassis_height" value="0.005" />
+    <xacro:property name="chassis_mass" value="0.2" />
     <!-- wheel properties -->
-    <xacro:property name="wheel_xoffset" value="0.048" />
     <xacro:property name="wheel_yoffset" value="0.095" />
-    <xacro:property name="wheel_zoffset" value="-0.013" />
     <xacro:property name="wheel_radius" value="0.0325" />
     <xacro:property name="wheel_width" value="0.027" />
     <xacro:property name="wheel_mass" value="0.032" />
     <!-- caster properties -->
-    <xacro:property name="caster_xoffset" value="-0.044" />
+    <xacro:property name="caster_xoffset" value="-0.092" />
     <xacro:property name="caster_radius" value="0.014" />
     <xacro:property name="caster_mass" value="0.05" />
@@ -29,5 +29,5 @@
             <parent link="base_link" />
             <child link="${prefix}_link" />
-            <origin xyz="${wheel_xoffset} ${y_reflect*wheel_yoffset} ${wheel_zoffset}" rpy="${-pi/2} 0 0" />
+            <origin xyz="0 ${y_reflect*wheel_yoffset} 0" rpy="${-pi/2} 0 0" />
             <axis xyz="0 0 1" />
         </joint>
@@ -50,9 +50,17 @@
         </gazebo>
     </xacro:macro>
-    <!-- BASE -->
+    <!-- DUMMY BASE -->
     <link name="base_link">
+    </link>
+    <!-- CHASSIS -->
+    <joint name="chassis_joint" type="fixed">
+        <parent link="base_link" />
+        <child link="chassis_link" />
+        <origin xyz="${chassis_xoffset} 0 ${chassis_zoffset}" />
+    </joint>
+    <link name="chassis_link">
         <visual>
             <geometry>
-                <box size="${base_depth} ${base_width} ${base_height}"/>
+                <box size="${chassis_depth} ${chassis_width} ${chassis_height}"/>
             </geometry>
             <material name="purple"/>
@@ -60,19 +68,19 @@
         <collision>
             <geometry>
-                <box size="${base_depth} ${base_width} ${base_height}"/>
+                <box size="${chassis_depth} ${chassis_width} ${chassis_height}"/>
             </geometry>
         </collision>
-        <xacro:box_inertia m="${base_mass}" x="${base_depth}" y="${base_width}" z="${base_height}" />
+        <xacro:box_inertia m="${chassis_mass}" x="${chassis_depth}" y="${chassis_width}" z="${chassis_height}" />
     </link>
-    <gazebo reference="base_link">
+    <gazebo reference="chassis_link">
         <material>Gazebo/Purple</material>
     </gazebo>
-    <joint name="caster_joint" type="fixed">
+    <!-- CASTER WHEEL -->
+    <!-- <joint name="caster_joint" type="fixed">
         <parent link="base_link" />
-        <child link="caster" />
-        <origin xyz="${caster_xoffset} 0.0 ${caster_radius-wheel_radius+wheel_zoffset}" />
+        <child link="caster_link" />
+        <origin xyz="${caster_xoffset} 0.0 ${caster_radius-wheel_radius}" />
     </joint>
-    <!-- CASTER WHEEL -->
-    <link name="caster">
+    <link name="caster_link">
         <visual>
             <geometry>
@@ -88,93 +96,11 @@
         <xacro:sphere_inertia m="${caster_mass}" r="${caster_radius}" />
     </link>
-    <gazebo reference="caster">
-        <mu1>0.0001</mu1>
-        <mu2>0.0001</mu2>
+    <gazebo reference="caster_link">
+        <mu1>0.00000001</mu1>
+        <mu2>0.00000001</mu2>
         <material>Gazebo/Gray</material>
-    </gazebo>
+    </gazebo> -->
     <!-- LEFT AND RIGHT WHEEL -->
-    <xacro:wheel prefix="left_wheel" y_reflect="1" />
-    <xacro:wheel prefix="right_wheel" y_reflect="-1" />
-    <gazebo>
-        <plugin name="differential_drive_controller" filename="libgazebo_ros_diff_drive.so">
-            <ros>
-                <namespace>/homeplater</namespace>
-                <!-- <argument>cmd_vel:=cmd_demo</argument>
-                <argument>odom:=odom_demo</argument> -->
-            </ros>
-            <!-- wheels -->
-            <left_joint>left_wheel_joint</left_joint>
-            <right_joint>right_wheel_joint</right_joint>
-            <!-- kinematics -->
-            <wheel_separation>0.19</wheel_separation>
-            <wheel_diameter>0.065</wheel_diameter>
-            <!-- tfs -->
-            <publish_odom>true</publish_odom>
-            <publish_odom_tf>true</publish_odom_tf>
-            <publish_wheel_tf>true</publish_wheel_tf>
-            <odometry_frame>odom</odometry_frame>
-            <!-- limits -->
-            <max_wheel_torque>20</max_wheel_torque>
-            <max_acceleration>1.0</max_acceleration>
-            <!-- miscs -->
-            <robot_base_frame>base_link</robot_base_frame>
-            <update_rate>50</update_rate>
-        </plugin>
-    </gazebo>
-    <!-- LIDAR -->
-    <joint name="lidar_joint" type="fixed">
-        <parent link="base_link" />
-        <child link="lidar" />
-        <origin xyz="0 0 ${(base_height+lidar_height)/2+lidar_zoff}" />
-    </joint>
-    <link name="lidar">
-        <visual>
-            <geometry>
-                <cylinder radius="${lidar_radius}" length="${lidar_height}" />
-            </geometry>
-            <material name="black" />
-        </visual>
-        <collision>
-            <origin xyz="0 0 0" rpy="0 0 0" />
-            <geometry>
-                <cylinder radius="${lidar_radius}" length="${lidar_height}" />
-            </geometry>
-        </collision>
-        <xacro:cylinder_inertia m="${lidar_mass}" r="${lidar_radius}" h="${lidar_height}" />
-    </link>
-    <gazebo reference="lidar">
-        <material>Gazebo/Black</material>
-        <sensor name="lidar" type="ray">
-            <always_on>true</always_on>
-            <visualize>true</visualize>
-            <update_rate>5</update_rate>
-            <ray>
-                <scan>
-                    <horizontal>
-                        <samples>360</samples>
-                        <resolution>1.000000</resolution>
-                        <min_angle>0.000000</min_angle>
-                        <max_angle>6.280000</max_angle>
-                    </horizontal>
-                </scan>
-                <range>
-                    <min>0.120000</min>
-                    <max>6</max>
-                    <resolution>0.015000</resolution>
-                </range>
-                <noise>
-                    <type>gaussian</type>
-                    <mean>0.0</mean>
-                    <stddev>0.01</stddev>
-                </noise>
-            </ray>
-            <plugin name="scan" filename="libgazebo_ros_ray_sensor.so">
-                <ros>
-                    <remapping>~/out:=scan</remapping>
-                </ros>
-                <output_type>sensor_msgs/LaserScan</output_type>
-                <frame_name>lidar</frame_name>
-            </plugin>
-        </sensor>
-    </gazebo>
+    <!-- <xacro:wheel prefix="left_wheel" y_reflect="1" />
+    <xacro:wheel prefix="right_wheel" y_reflect="-1" /> -->
 </robot>

Commit message: include slam_toolbox

File: hpr_description/urdf/hpr_core.urdf.xacro (robot description, xacro)
@@ -78,4 +78,12 @@
         <material>Gazebo/Purple</material>
     </gazebo>
+    <!-- FOOTPRINT -->
+    <joint name="footprint_joint" type="fixed">
+        <parent link="base_link" />
+        <child link="base_footprint" />
+        <origin xyz="${chassis_xoffset} 0 ${-wheel_radius}" />
+    </joint>
+    <link name="base_footprint">
+    </link>
     <!-- CASTER WHEEL -->
     <joint name="caster_joint" type="fixed">

Commit message: add launch file

File: hpr_description/urdf/hpr_core.urdf.xacro (robot description, xacro)
@@ -55,4 +55,12 @@
     <link name="base_link">
     </link>
+    <!-- FOOTPRINT -->
+    <joint name="footprint_joint" type="fixed">
+        <parent link="base_link" />
+        <child link="base_footprint" />
+        <origin xyz="${chassis_xoffset} 0 ${-wheel_radius}" />
+    </joint>
+    <link name="base_footprint">
+    </link>
     <!-- CHASSIS -->
     <joint name="chassis_joint" type="fixed">
@@ -78,5 +86,4 @@
         <material>Gazebo/Purple</material>
     </gazebo>
-<<<<<<< HEAD
     <!-- CASTER WHEEL -->
     <joint name="caster_joint" type="fixed">
@@ -85,20 +92,4 @@
         <origin xyz="${caster_xoffset} 0.0 ${caster_radius-wheel_radius}" />
     </joint>
-=======
-    <!-- FOOTPRINT -->
-    <joint name="footprint_joint" type="fixed">
-        <parent link="base_link" />
-        <child link="base_footprint" />
-        <origin xyz="${chassis_xoffset} 0 ${-wheel_radius}" />
-    </joint>
-    <link name="base_footprint">
-    </link>
-    <!-- CASTER WHEEL -->
-    <joint name="caster_joint" type="fixed">
-        <parent link="base_link" />
-        <child link="caster_link" />
-        <origin xyz="${caster_xoffset} 0.0 ${caster_radius-wheel_radius}" />
-    </joint>
->>>>>>> 7-sim_slam
     <link name="caster_link">
         <visual>
